File: pcb/neuropixels-2.0.kicad_sch (KiCad schematic)
At the start: 8 parts, among them J2 2013496-9, J3 2013496-9, U4 TS5A3159A, U5 DSC6011JI1A-048.0000

Commit message: Inital routing complete
- Addressed Aaron's review
- Pullup on output side of analog switch to prevent floating SDA
- Other minor changes
Parts:
- added C12: 0.1uF, Capacitor_SMD:C_0201_0603Metric, symbol Device:C
- added R1, R2 (x2): 1k, Resistor_SMD:R_0201_0603Metric, symbol Device:R_US
- renumbered C24 to C23, C25 to C24, J2 to J3, J3 to J4
Connections:
- net +1.8VA: now also R1.1, R2.1, R2.1
- net +1V8: now also C12.1
- net GND: now also C12.2
- net SCL: now also R1.2
- net SDA_{A}: now also R2.2
- net SDA_{B}: now also R2.2
Other:
- note added: "NB: 1.8VA is last rail to come up."
- note added: "NB: Effectively add another bit to device address (using NP_{Select}) so that two probes with the same address can be accessed sequentially."
- note added: "NB: This filter is used on the IMEC design. Maybe to reduce noise in the probe?. In anycase, easy to remove."
- moved on the sheet: U4

Commit message: Address team comments
- Add extra mouse-bite supports
- Enbiggen cable strain relief spear
- Add DNP 0.1" header for bench debug
- Small routing changes
- Update and complete BOM
Parts:
- C12: CASE/PACKAGE (none) -> 0201; Voltage 16V -> 25V
- C23, C24: CASE/PACKAGE (none) -> 0201
- R1, R2, R3, R4: CASE/PACKAGE (none) -> 0201; Tolerance (none) -> 1%
- renumbered J3 to J2, J4 to J3

Commit message: Updates to design after feedback from assembler
- Replace obsolete TE_2013496-9 ZIF connector used by IMEC with
046844727002846+, which should fit NP 2.0 flex connectors (see design
folder for comparison). We will see.
- Replaced programmable MEMS oscillator with standard quartz since this
is a common frequency.
- Other BOM updates to account for obsolete or out of stock components
Parts:
- J2, J3: value 2013496-9 -> 046844727002846+; footprint jonnew:TE_2013496-9 -> jonnew:KYOCERA_046844727002846+
- U4: value TS5A3159A -> TS5A3159AYZPR
- U5: value DSC6011JI1A-048.0000 -> ECS-2016MV-480-CN-TR; footprint jonnew:MICROCHIP_VFLGA4-2.0x1.6 -> jonnew:ECS_2016MV
Changed lines of the file:
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@@
       (effects (font (size 1.27 1.27)))
     )
-    (property "Value" "TS5A3159A" (at 74.93 83.82 0)
+    (property "Value" "TS5A3159AYZPR " (at 74.93 83.82 0)
       (effects (font (size 1.27 1.27)))
     )
@@
       (effects (font (size 1.27 1.27)))
     )
-    (property "Value" "2013496-9" (at 168.91 21.59 0)
-      (effects (font (size 1.27 1.27)))
-    )
-    (property "Footprint" "jonnew:TE_2013496-9" (at 168.91 40.64 0)
+    (property "Value" "046844727002846+" (at 168.91 21.59 0)
+      (effects (font (size 1.27 1.27)))
+    )
+    (property "Footprint" "jonnew:KYOCERA_046844727002846+" (at 168.91 40.64 0)
       (effects (font (size 1.27 1.27)) hide)
     )
@@
       (effects (font (size 1.27 1.27)))
     )
-    (property "Value" "2013496-9" (at 168.91 83.82 0)
-      (effects (font (size 1.27 1.27)))
-    )
-    (property "Footprint" "jonnew:TE_2013496-9" (at 168.91 102.87 0)
+    (property "Value" "046844727002846+" (at 168.91 83.82 0)
+      (effects (font (size 1.27 1.27)))
+    )
+    (property "Footprint" "jonnew:KYOCERA_046844727002846+" (at 168.91 102.87 0)
       (effects (font (size 1.27 1.27)) hide)
     )
@@
       (effects (font (size 1.27 1.27)))
     )
-    (property "Value" "DSC6011JI1A-048.0000" (at 168.91 144.78 0)
-      (effects (font (size 1.27 1.27)))
-    )
-    (property "Footprint" "jonnew:MICROCHIP_VFLGA4-2.0x1.6" (at 168.91 160.655 0)
-      (effects (font (size 1.27 1.27)) hide)
-    )
+    (property "Value" "ECS-2016MV-480-CN-TR" (at 168.91 144.78 0)
+      (effects (font (size 1.27 1.27)))
+    )
+    (property "Footprint" "jonnew:ECS_2016MV" (at 168.91 160.655 0)
+      (effects (font (size 1.27 1.27)) hide)
+    )
