File: pcb/neuropixels-2.0.kicad_sch (KiCad schematic)
At the start: 12 parts, among them J2 FH35C-17S-0.3SHW(99), J3 FH35C-17S-0.3SHW(99), U4 STG3856, U5 ECS-2016MV-480-CN-TR

Commit message: Added new fields (OEPS PN, MPN, and Type) to all components.
Parts:
- C12: MPN (none) -> GRM033R61E104KE14J; OEPS PN ?? -> OEPS010035; Type (none) -> SMD
- C23: MPN (none) -> GRM033R71E103KE14D; OEPS PN ?? -> OEPS010037; Type (none) -> SMD
- C24: MPN (none) -> GRM0335C1H270GA01D; OEPS PN ?? -> OEPS010029; Type (none) -> SMD
- J2, J3: MPN (none) -> FH35C-17S-0.3SHW(99); OEPS PN ?? -> OEPS070073; Type (none) -> SMD
- R2: MPN (none) -> CRCW020110K0FNED; OEPS PN ?? -> OEPS020066; Type (none) -> SMD
- R4: MPN (none) -> RC0201FR-0710RL; OEPS PN ?? -> OEPS020084; Type (none) -> SMD
- U4: MPN (none) -> STG3856QTR; OEPS PN ?? -> OEPS080088; Type (none) -> SMD
- U5: MPN (none) -> ECS-2016MV-480-CN-TR; OEPS PN ?? -> OEPS080079; Type (none) -> SMD
Changed lines of the file:
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@@
       (effects (font (size 1.27 1.27)) hide)
     )
-    (property "OEPS PN" "??" (at 67.31 97.79 0)
+    (property "OEPS PN" "OEPS080088" (at 67.31 97.79 0)
+      (effects (font (size 1.27 1.27)) hide)
+    )
+    (property "MPN" "STG3856QTR" (at 67.31 97.79 0)
+      (effects (font (size 1.27 1.27)) hide)
+    )
+    (property "Type" "SMD" (at 67.31 97.79 0)
       (effects (font (size 1.27 1.27)) hide)
     )
@@
       (effects (font (size 1.27 1.27)) hide)
     )
-    (property "OEPS PN" "??" (at 107.95 78.74 0)
+    (property "OEPS PN" "OEPS020066" (at 107.95 78.74 0)
+      (effects (font (size 1.27 1.27)) hide)
+    )
+    (property "MPN" "CRCW020110K0FNED" (at 107.95 78.74 0)
+      (effects (font (size 1.27 1.27)) hide)
+    )
+    (property "Type" "SMD" (at 107.95 78.74 0)
       (effects (font (size 1.27 1.27)) hide)
     )
@@
       (effects (font (size 1.27 1.27)) hide)
     )
-    (property "OEPS PN" "??" (at 191.77 148.59 0)
+    (property "OEPS PN" "OEPS020084" (at 191.77 148.59 0)
+      (effects (font (size 1.27 1.27)) hide)
+    )
+    (property "MPN" "RC0201FR-0710RL" (at 191.77 148.59 0)
+      (effects (font (size 1.27 1.27)) hide)
+    )
+    (property "Type" "SMD" (at 191.77 148.59 0)
       (effects (font (size 1.27 1.27)) hide)
     )
@@
       (effects (font (size 1.27 1.27)) hide)
     )
-    (property "OEPS PN" "??" (at 116.84 78.74 0)
+    (property "OEPS PN" "OEPS020066" (at 116.84 78.74 0)
+      (effects (font (size 1.27 1.27)) hide)
+    )
+    (property "MPN" "CRCW020110K0FNED" (at 116.84 78.74 0)
+      (effects (font (size 1.27 1.27)) hide)
+    )
+    (property "Type" "SMD" (at 116.84 78.74 0)
       (effects (font (size 1.27 1.27)) hide)
     )
@@
       (effects (font (size 1.27 1.27)) hide)
     )
-    (property "OEPS PN" "??" (at 199.39 153.67 0)
+    (property "OEPS PN" "OEPS010029" (at 199.39 153.67 0)
+      (effects (font (size 1.27 1.27)) hide)
+    )
+    (property "MPN" "GRM0335C1H270GA01D" (at 199.39 153.67 0)
+      (effects (font (size 1.27 1.27)) hide)
+    )
+    (property "Type" "SMD" (at 199.39 153.67 0)
       (effects (font (size 1.27 1.27)) hide)
     )
@@
       (effects (font (size 1.27 1.27)) hide)
     )
-    (property "OEPS PN" "??" (at 147.32 153.67 0)
+    (property "OEPS PN" "OEPS010037" (at 147.32 153.67 0)
+      (effects (font (size 1.27 1.27)) hide)
+    )
+    (property "MPN" "GRM033R71E103KE14D" (at 147.32 153.67 0)
+      (effects (font (size 1.27 1.27)) hide)
+    )
+    (property "Type" "SMD" (at 147.32 153.67 0)
       (effects (font (size 1.27 1.27)) hide)
     )
@@
       (effects (font (size 1.27 1.27)) hide)
     )
-    (property "OEPS PN" "??" (at 99.06 78.74 0)
+    (property "OEPS PN" "OEPS020066" (at 99.06 78.74 0)
+      (effects (font (size 1.27 1.27)) hide)
+    )
+    (property "MPN" "CRCW020110K0FNED" (at 99.06 78.74 0)
+      (effects (font (size 1.27 1.27)) hide)
+    )
+    (property "Type" "SMD" (at 99.06 78.74 0)
       (effects (font (size 1.27 1.27)) hide)
     )
@@
       (effects (font (size 1.27 1.27)) hide)
     )
-    (property "OEPS PN" "??" (at 90.17 78.74 0)
+    (property "OEPS PN" "OEPS020066" (at 90.17 78.74 0)
+      (effects (font (size 1.27 1.27)) hide)
+    )
+    (property "MPN" "CRCW020110K0FNED" (at 90.17 78.74 0)
+      (effects (font (size 1.27 1.27)) hide)
+    )
+    (property "Type" "SMD" (at 90.17 78.74 0)
       (effects (font (size 1.27 1.27)) hide)
     )
@@
       (effects (font (size 1.27 1.27)) hide)
     )
-    (property "OEPS PN" "??" (at 36.83 95.25 0)
+    (property "OEPS PN" "OEPS010035" (at 36.83 95.25 0)
+      (effects (font (size 1.27 1.27)) hide)
+    )
+    (property "MPN" "GRM033R61E104KE14J" (at 36.83 95.25 0)
+      (effects (font (size 1.27 1.27)) hide)
+    )
+    (property "Type" "SMD" (at 36.83 95.25 0)
       (effects (font (size 1.27 1.27)) hide)
     )
@@
       (effects (font (size 1.27 1.27)) hide)
     )
-    (property "OEPS PN" "??" (at 171.45 104.14 0)
+    (property "OEPS PN" "OEPS070073" (at 171.45 104.14 0)
+      (effects (font (size 1.27 1.27)) hide)
+    )
+    (property "MPN" "FH35C-17S-0.3SHW(99)" (at 171.45 104.14 0)
+      (effects (font (size 1.27 1.27)) hide)
+    )
+    (property "Type" "SMD" (at 171.45 104.14 0)
       (effects (font (size 1.27 1.27)) hide)
     )
@@
       (effects (font (size 1.27 1.27)) hide)
     )
-    (property "OEPS PN" "??" (at 171.45 151.13 0)
+    (property "OEPS PN" "OEPS080079" (at 171.45 151.13 0)
+      (effects (font (size 1.27 1.27)) hide)
+    )
+    (property "MPN" "ECS-2016MV-480-CN-TR" (at 171.45 151.13 0)
+      (effects (font (size 1.27 1.27)) hide)
+    )
+    (property "Type" "SMD" (at 171.45 151.13 0)
       (effects (font (size 1.27 1.27)) hide)
     )
@@
       (effects (font (size 1.27 1.27)) hide)
     )
-    (property "OEPS PN" "??" (at 171.45 44.45 0)
-      (effects (font (size 1.27 1.27)) hide)
-    )
+    (property "OEPS PN" "OEPS070073" (at 171.45 44.45 0)
+      (effects (font (size 1.27 1.27)) hide)
+    )
+    (property "MPN" "FH35C-17S-0.3SHW(99)" (at 171.45 44.45 0)
+      (effects (font (size 1.27 1.27)) hide)
+    )
+    (property "Type" "SMD" (at 171.45 44.45 0)
+      (effects (font (size 1.27 1.27)) hide)
+    )
