File: pcb/power.kicad_sch (KiCad schematic)
At the start: 11 parts, among them U1 MIC5335-JGYMT, U2 NCP163AFCT180T2G

Commit message: Revision B
- Fix incorrect STG3856 symbol and make corresponding changes to PCB
- Flip bits 1 and 2 in probe interaces (fixes #1)
- Improve silkscreen
Parts:
- C12, L1, L2, R3, R4, U1, U2: OEPS PN (none) -> ??
Changed lines of the file:
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@@
     (title "ONIX Neuropixels 2.0 Economical Headstage")
     (date "2021-12-16")
-    (rev "A")
+    (rev "B")
     (company "Open Ephys, Inc")
     (comment 1 "Jonathan P. Newman")
@@
       (effects (font (size 1.27 1.27)) hide)
     )
+    (property "OEPS PN" "" (at 152.4 124.46 0)
+      (effects (font (size 1.27 1.27)) hide)
+    )
     (pin "1")
     (pin "2")
@@
       (effects (font (size 1.27 1.27)) hide)
     )
+    (property "OEPS PN" "??" (at 207.01 72.39 0)
+      (effects (font (size 1.27 1.27)) hide)
+    )
     (pin "1")
     (pin "2")
@@
     )
     (property "Tolerance" "" (at 130.81 66.04 0)
+      (effects (font (size 1.27 1.27)) hide)
+    )
+    (property "OEPS PN" "??" (at 130.81 66.04 0)
       (effects (font (size 1.27 1.27)) hide)
     )
@@
       (effects (font (size 1.27 1.27)) hide)
     )
+    (property "OEPS PN" "" (at 114.3 76.2 0)
+      (effects (font (size 1.27 1.27)) hide)
+    )
     (pin "1")
     (pin "2")
@@
       (effects (font (size 1.27 1.27)) hide)
     )
+    (property "OEPS PN" "" (at 100.33 124.46 0)
+      (effects (font (size 1.27 1.27)) hide)
+    )
     (pin "1")
     (pin "2")
@@
     )
     (property "Tolerance" "" (at 97.79 76.2 0)
+      (effects (font (size 1.27 1.27)) hide)
+    )
+    (property "OEPS PN" "" (at 97.79 76.2 0)
       (effects (font (size 1.27 1.27)) hide)
     )
@@
       (effects (font (size 1.27 1.27)) hide)
     )
+    (property "OEPS PN" "??" (at 189.23 63.5 0)
+      (effects (font (size 1.27 1.27)) hide)
+    )
     (pin "1")
     (pin "2")
@@
     )
     (property "Tolerance" "" (at 127 119.38 0)
+      (effects (font (size 1.27 1.27)) hide)
+    )
+    (property "OEPS PN" "??" (at 127 119.38 0)
       (effects (font (size 1.27 1.27)) hide)
     )
@@
       (effects (font (size 1.27 1.27)) hide)
     )
+    (property "OEPS PN" "??" (at 207.01 63.5 0)
+      (effects (font (size 1.27 1.27)) hide)
+    )
     (pin "1")
     (pin "2")
@@
       (effects (font (size 1.27 1.27)) hide)
     )
+    (property "OEPS PN" "??" (at 152.4 76.2 0)
+      (effects (font (size 1.27 1.27)) hide)
+    )
     (pin "1")
     (pin "2")
@@
       (effects (font (size 1.27 1.27)) hide)
     )
+    (property "OEPS PN" "??" (at 189.23 72.39 0)
+      (effects (font (size 1.27 1.27)) hide)
+    )

Commit message: Added new fields (OEPS PN, MPN, and Type) to all components.
Parts:
- C1, C2, C4, C5: MPN (none) -> CL03A105MO3NRNH; OEPS PN (none) -> OEPS010036; Type (none) -> SMD
- C12: MPN (none) -> CL05A106MP5NUNC; OEPS PN ?? -> OEPS010038; Type (none) -> SMD
- L1: MPN (none) -> CBC3225T101MR; OEPS PN ?? -> OEPS040010; Type (none) -> SMD
- L2: MPN (none) -> ASMPH-0805-4R7M-T; OEPS PN ?? -> OEPS040007; Type (none) -> SMD
- R3, R4: MPN (none) -> RC0201FR-072KL; OEPS PN ?? -> OEPS020067; Type (none) -> SMD
- U1: MPN (none) -> MIC5335-JGYMT; OEPS PN ?? -> OEPS080045; Type (none) -> SMD
- U2: MPN (none) -> NCP163AFCT180T2G; OEPS PN ?? -> OEPS080077; Type (none) -> SMD
Changed lines of the file:
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@@
       (effects (font (size 1.27 1.27)) hide)
     )
-    (property "OEPS PN" "" (at 152.4 124.46 0)
+    (property "OEPS PN" "OEPS010036" (at 152.4 124.46 0)
+      (effects (font (size 1.27 1.27)) hide)
+    )
+    (property "MPN" "CL03A105MO3NRNH" (at 152.4 124.46 0)
+      (effects (font (size 1.27 1.27)) hide)
+    )
+    (property "Type" "SMD" (at 152.4 124.46 0)
       (effects (font (size 1.27 1.27)) hide)
     )
@@
       (effects (font (size 1.27 1.27)) hide)
     )
-    (property "OEPS PN" "??" (at 207.01 72.39 0)
+    (property "OEPS PN" "OEPS040007" (at 207.01 72.39 0)
+      (effects (font (size 1.27 1.27)) hide)
+    )
+    (property "MPN" "ASMPH-0805-4R7M-T" (at 207.01 72.39 0)
+      (effects (font (size 1.27 1.27)) hide)
+    )
+    (property "Type" "SMD" (at 207.01 72.39 0)
       (effects (font (size 1.27 1.27)) hide)
     )
@@
       (effects (font (size 1.27 1.27)) hide)
     )
-    (property "OEPS PN" "??" (at 130.81 66.04 0)
+    (property "OEPS PN" "OEPS080045" (at 130.81 66.04 0)
+      (effects (font (size 1.27 1.27)) hide)
+    )
+    (property "MPN" "MIC5335-JGYMT" (at 130.81 66.04 0)
+      (effects (font (size 1.27 1.27)) hide)
+    )
+    (property "Type" "SMD" (at 130.81 66.04 0)
       (effects (font (size 1.27 1.27)) hide)
     )
@@
       (effects (font (size 1.27 1.27)) hide)
     )
-    (property "OEPS PN" "" (at 114.3 76.2 0)
+    (property "OEPS PN" "OEPS010036" (at 114.3 76.2 0)
+      (effects (font (size 1.27 1.27)) hide)
+    )
+    (property "MPN" "CL03A105MO3NRNH" (at 114.3 76.2 0)
+      (effects (font (size 1.27 1.27)) hide)
+    )
+    (property "Type" "SMD" (at 114.3 76.2 0)
       (effects (font (size 1.27 1.27)) hide)
     )
@@
       (effects (font (size 1.27 1.27)) hide)
     )
-    (property "OEPS PN" "" (at 100.33 124.46 0)
+    (property "OEPS PN" "OEPS010036" (at 100.33 124.46 0)
+      (effects (font (size 1.27 1.27)) hide)
+    )
+    (property "MPN" "CL03A105MO3NRNH" (at 100.33 124.46 0)
+      (effects (font (size 1.27 1.27)) hide)
+    )
+    (property "Type" "SMD" (at 100.33 124.46 0)
       (effects (font (size 1.27 1.27)) hide)
     )
@@
       (effects (font (size 1.27 1.27)) hide)
     )
-    (property "OEPS PN" "" (at 97.79 76.2 0)
+    (property "OEPS PN" "OEPS010036" (at 97.79 76.2 0)
+      (effects (font (size 1.27 1.27)) hide)
+    )
+    (property "MPN" "CL03A105MO3NRNH" (at 97.79 76.2 0)
+      (effects (font (size 1.27 1.27)) hide)
+    )
+    (property "Type" "SMD" (at 97.79 76.2 0)
       (effects (font (size 1.27 1.27)) hide)
     )
@@
       (effects (font (size 1.27 1.27)) hide)
     )
-    (property "OEPS PN" "??" (at 189.23 63.5 0)
+    (property "OEPS PN" "OEPS020067" (at 189.23 63.5 0)
+      (effects (font (size 1.27 1.27)) hide)
+    )
+    (property "MPN" "RC0201FR-072KL" (at 189.23 63.5 0)
+      (effects (font (size 1.27 1.27)) hide)
+    )
+    (property "Type" "SMD" (at 189.23 63.5 0)
       (effects (font (size 1.27 1.27)) hide)
     )
@@
       (effects (font (size 1.27 1.27)) hide)
     )
-    (property "OEPS PN" "??" (at 127 119.38 0)
+    (property "OEPS PN" "OEPS080077" (at 127 119.38 0)
+      (effects (font (size 1.27 1.27)) hide)
+    )
+    (property "MPN" "NCP163AFCT180T2G" (at 127 119.38 0)
+      (effects (font (size 1.27 1.27)) hide)
+    )
+    (property "Type" "SMD" (at 127 119.38 0)
       (effects (font (size 1.27 1.27)) hide)
     )
@@
       (effects (font (size 1.27 1.27)) hide)
     )
-    (property "OEPS PN" "??" (at 207.01 63.5 0)
+    (property "OEPS PN" "OEPS020067" (at 207.01 63.5 0)
+      (effects (font (size 1.27 1.27)) hide)
+    )
+    (property "MPN" "RC0201FR-072KL" (at 207.01 63.5 0)
+      (effects (font (size 1.27 1.27)) hide)
+    )
+    (property "Type" "SMD" (at 207.01 63.5 0)
       (effects (font (size 1.27 1.27)) hide)
     )
@@
       (effects (font (size 1.27 1.27)) hide)
     )
-    (property "OEPS PN" "??" (at 152.4 76.2 0)
+    (property "OEPS PN" "OEPS010038" (at 152.4 76.2 0)
+      (effects (font (size 1.27 1.27)) hide)
+    )
+    (property "MPN" "CL05A106MP5NUNC" (at 152.4 76.2 0)
+      (effects (font (size 1.27 1.27)) hide)
+    )
+    (property "Type" "SMD" (at 152.4 76.2 0)
       (effects (font (size 1.27 1.27)) hide)
     )
@@
       (effects (font (size 1.27 1.27)) hide)
     )
-    (property "OEPS PN" "??" (at 189.23 72.39 0)
-      (effects (font (size 1.27 1.27)) hide)
-    )
+    (property "OEPS PN" "OEPS040010" (at 189.23 72.39 0)
+      (effects (font (size 1.27 1.27)) hide)
+    )
+    (property "MPN" "CBC3225T101MR" (at 189.23 72.39 0)
+      (effects (font (size 1.27 1.27)) hide)
+    )
+    (property "Type" "SMD" (at 189.23 72.39 0)
+      (effects (font (size 1.27 1.27)) hide)
+    )
