File: pcb/serializer.kicad_sch (KiCad schematic)
At the start: 23 parts, among them U3 DS90UB933TRTVTQ1

Commit message: Revision B
- Fix incorrect STG3856 symbol and make corresponding changes to PCB
- Flip bits 1 and 2 in probe interaces (fixes #1)
- Improve silkscreen
Parts:
- C10, C11, C12, C13, C14, C15, C16, C17, C18, C19, C20, C6, C7, C8, C9, L3, L4, R5, R6, R7, R8, U3: OEPS PN (none) -> ??
Connections:
- net D1_{A}: now also U3.31 (DIN_10); no longer U3.29 (DIN_8)
- net D1_{B}: now also U3.27 (DIN_7); no longer U3.30 (DIN_9)
- net D2_{A}: now also U3.29 (DIN_8); no longer U3.31 (DIN_10)
- net D2_{B}: now also U3.30 (DIN_9); no longer U3.27 (DIN_7)
Other:
- moved on the sheet: C21, R6, R7

Commit message: Added new fields (OEPS PN, MPN, and Type) to all components.
Parts:
- C10, C13, C16, C6, C8: MPN (none) -> GRM033R71E103KE14D; OEPS PN ?? -> OEPS010037; Type (none) -> SMD
- C11, C14, C17, C19, C7, C9: MPN (none) -> GRM033R61E104KE14J; OEPS PN ?? -> OEPS010035; Type (none) -> SMD
- C12, C15, C18: MPN (none) -> CL05A106MP5NUNC; OEPS PN ?? -> OEPS010038; Type (none) -> SMD
- C20: MPN (none) -> CC0201KRX5R8BB473; OEPS PN ?? -> OEPS010031; Type (none) -> SMD
- C21: MPN (none) -> CL03A105MO3NRNH; OEPS PN (none) -> OEPS010036; Type (none) -> SMD
- L3, L4: MPN (none) -> BLF03RD501GZED; OEPS PN ?? -> OEPS040006; Type (none) -> SMD
- R5, R6, R7: MPN (none) -> CRCW020110K0FNED; OEPS PN ?? -> OEPS020066; Type (none) -> SMD
- R8: MPN (none) -> RC0201FR-0749R9L; OEPS PN ?? -> OEPS020068; Type (none) -> SMD
- U3: MPN (none) -> DS90UB933TRTVTQ1; OEPS PN ?? -> OEPS080064; Type (none) -> SMD
