File: pcb/headstage-neuropix2e.kicad_pcb (KiCad board)
At the start: 4 copper layers, 60 x 60 mm, 64 parts, among them J1 X.FL-R-SMT-1(02), J2 FH35C-17S-0.3SHW(99), J3 FH35C-17S-0.3SHW(99), J4 SBH11-PBPC-D05-ST-BK, J5 TC2030, J6 050700622, U1 MIC5335-JGYMT, U2 NCP163AFCT180T2G, U3 DS90UB933TRTVTQ1, U4 STG3856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

Commit message: Revision B
- Fix incorrect STG3856 symbol and make corresponding changes to PCB
- Flip bits 1 and 2 in probe interaces (fixes #1)
- Improve silkscreen
Parts:
- TP2: value NP_{TP0} -> NP_{Lesion}
- TP3: value NP_{TP1} -> NP_{Cal}
- moved R10 7.97 mm to (146.4, 92.6)
- moved R12 7.96 mm to (138.6, 93.9)
- moved R11 7.85 mm to (146.4, 92.6)
- moved R9 7.85 mm to (138.6, 92.5)
- moved C22 2.55 mm to (146.4, 89.4), turned to -90 degrees
- moved U4 0.68 mm to (144.8, 89.3), turned to -90 degrees
Connections:
- net /Neuropixels 2.0/NP_{TP0} renamed /Neuropixels 2.0/NP_{Lesion}
- net /Neuropixels 2.0/NP_{TP1} renamed /Neuropixels 2.0/NP_{Cal}
- net /Neuropixels 2.0/NP_{~{MUXRST}} renamed /Neuropixels 2.0/NP_{~{RST}}
- J2 pad 11: /Neuropixels 2.0/D2_{A} -> /Neuropixels 2.0/D1_{A}
- J2 pad 7: /Neuropixels 2.0/D1_{A} -> /Neuropixels 2.0/D2_{A}
- J3 pad 11: /Neuropixels 2.0/D2_{B} -> /Neuropixels 2.0/D1_{B}
- J3 pad 7: /Neuropixels 2.0/D1_{B} -> /Neuropixels 2.0/D2_{B}
- R10 pad 2: /Neuropixels 2.0/SCL_{B} -> /Neuropixels 2.0/SDA_{B}
- R11 pad 2: /Neuropixels 2.0/SDA_{A} -> /Neuropixels 2.0/SCL_{A}
- R12 pad 2: /Neuropixels 2.0/SDA_{B} -> /Neuropixels 2.0/SCL_{B}
- R5 pad 1: /Neuropixels 2.0/NP_{Sel1} -> /Neuropixels 2.0/NP_{Sel0}
- R9 pad 2: /Neuropixels 2.0/SCL_{A} -> /Neuropixels 2.0/SDA_{A}
- U3 pad 17: /Neuropixels 2.0/NP_{Sel1} -> /Neuropixels 2.0/NP_{Sel0}
- U3 pad 18: /Neuropixels 2.0/NP_{Sel0} -> /Neuropixels 2.0/NP_{Sel1}
- U3 pad 27: /Neuropixels 2.0/D2_{B} -> /Neuropixels 2.0/D1_{B}
- U3 pad 29: /Neuropixels 2.0/D1_{A} -> /Neuropixels 2.0/D2_{A}
- U3 pad 30: /Neuropixels 2.0/D1_{B} -> /Neuropixels 2.0/D2_{B}
- U3 pad 31: /Neuropixels 2.0/D2_{A} -> /Neuropixels 2.0/D1_{A}
- U4 pad 10: /Neuropixels 2.0/SDA -> /Neuropixels 2.0/NP_{Sel1}
- U4 pad 12: /Neuropixels 2.0/SCL -> /Neuropixels 2.0/NP_{Sel0}
- U4 pad 2: /Neuropixels 2.0/SCL_{A} -> /Neuropixels 2.0/SDA_{A}
- U4 pad 3: /Neuropixels 2.0/SCL_{B} -> /Neuropixels 2.0/SDA_{B}
- U4 pad 4: /Neuropixels 2.0/NP_{Sel0} -> /Neuropixels 2.0/SDA
- U4 pad 6: /Neuropixels 2.0/NP_{Sel1} -> /Neuropixels 2.0/SCL
- U4 pad 7: /Neuropixels 2.0/SDA_{B} -> /Neuropixels 2.0/SCL_{B}
- U4 pad 8: /Neuropixels 2.0/SDA_{A} -> /Neuropixels 2.0/SCL_{A}
Routing:
- net /Neuropixels 2.0/SCL_{B}: track 11.1 -> 9.61 mm
- net /Neuropixels 2.0/NP_{Sel1}: track 3.78 -> 5.19 mm
- net /Neuropixels 2.0/SDA_{A}: track 11.2 -> 12.5 mm
- net /Neuropixels 2.0/SCL: track 59.2 -> 58.1 mm
- net +1V8: track 35.6 -> 34.5 mm
- net /Neuropixels 2.0/NP_{Sel0}: track 3.01 -> 4.08 mm, vias 1 -> 2
- net /Neuropixels 2.0/SDA_{B}: track 11.8 -> 12.7 mm
- net GND: vias 66 -> 73
Other:
- outline, holes or cut-outs redrawn
- board text added: "2.7V ≤ V_{coax} ≥ 5.5V"
- board text added: "C"
- board text added: "ONIX Headstage Neuropix-2.0e (Public) Board Rev. B"
- board text added: "V_{coax}"
- board text added: "rB"
- board text removed: "+3V"
- board text removed: "1"
- board text removed: "ONIX Headstage Neuropix-2.0e (Public) Board Rev. A"
- board text removed: "rA"
