File: pcb/perpherials.kicad_sch (KiCad schematic)
At the start: 9 parts, among them J4 TC2030, J6 050700622, J6 SBH11-PBPC-D05-ST-BK, U6 M24C64-FCS6TP/K, U7 BNO055

Commit message: Changed expansion's (J6) attribute to be part of the BOM.
Parts:
- J6: now in the parts list
Changed lines of the file:
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@@
   )
   (symbol (lib_id "jonnew:Conn_02x3_Odd_Even_4Mech") (at 214.63 125.73 0) (unit 1)
-    (in_bom no) (on_board yes) (dnp no)
+    (in_bom yes) (on_board yes) (dnp no)
     (property "Reference" "J6" (at 214.63 114.3 0)
       (effects (font (size 1.27 1.27)))

Commit message: Added new fields (OEPS PN, MPN, and Type) to all components.
Parts:
- C25, C26, C27, C28: MPN (none) -> GRM033R61E104KE14J; OEPS PN ?? -> OEPS010035; Type (none) -> SMD
- J4: MPN (none) -> -; OEPS PN ?? -> -; Type (none) -> -
- J6: OEPS PN ?? -> OEPS070049
- J6: MPN (none) -> SBH11-PBPC-D05-ST-BK; OEPS PN ?? -> OEPS070030; Type (none) -> TH
- U6: MPN (none) -> M24C64-FCS6TP/K; OEPS PN ?? -> OEPS080050; Type (none) -> SMD
- U7: MPN (none) -> BNO055; OEPS PN ?? -> OEPS080063; Type (none) -> SMD
Changed lines of the file:
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@@
       (effects (font (size 1.27 1.27)) hide)
     )
-    (property "OEPS PN" "??" (at 129.54 127 0)
+    (property "OEPS PN" "OEPS080063" (at 129.54 127 0)
+      (effects (font (size 1.27 1.27)) hide)
+    )
+    (property "MPN" "BNO055" (at 129.54 127 0)
+      (effects (font (size 1.27 1.27)) hide)
+    )
+    (property "Type" "SMD" (at 129.54 127 0)
       (effects (font (size 1.27 1.27)) hide)
     )
@@
       (effects (font (size 1.27 1.27)) hide)
     )
-    (property "OEPS PN" "??" (at 214.63 125.73 0)
+    (property "OEPS PN" "OEPS070049" (at 214.63 125.73 0)
       (effects (font (size 1.27 1.27)) hide)
     )
@@
       (effects (font (size 1.27 1.27)) hide)
     )
-    (property "OEPS PN" "??" (at 217.17 59.69 0)
+    (property "OEPS PN" "OEPS010035" (at 217.17 59.69 0)
+      (effects (font (size 1.27 1.27)) hide)
+    )
+    (property "MPN" "GRM033R61E104KE14J" (at 217.17 59.69 0)
+      (effects (font (size 1.27 1.27)) hide)
+    )
+    (property "Type" "SMD" (at 217.17 59.69 0)
       (effects (font (size 1.27 1.27)) hide)
     )
@@
       (effects (font (size 1.27 1.27)) hide)
     )
-    (property "OEPS PN" "??" (at 198.12 59.69 0)
+    (property "OEPS PN" "OEPS080050" (at 198.12 59.69 0)
+      (effects (font (size 1.27 1.27)) hide)
+    )
+    (property "MPN" "M24C64-FCS6TP/K" (at 198.12 59.69 0)
+      (effects (font (size 1.27 1.27)) hide)
+    )
+    (property "Type" "SMD" (at 198.12 59.69 0)
       (effects (font (size 1.27 1.27)) hide)
     )
@@
       (effects (font (size 1.27 1.27)) hide)
     )
-    (property "OEPS PN" "??" (at 87.63 110.49 0)
+    (property "OEPS PN" "OEPS010035" (at 87.63 110.49 0)
+      (effects (font (size 1.27 1.27)) hide)
+    )
+    (property "MPN" "GRM033R61E104KE14J" (at 87.63 110.49 0)
+      (effects (font (size 1.27 1.27)) hide)
+    )
+    (property "Type" "SMD" (at 87.63 110.49 0)
       (effects (font (size 1.27 1.27)) hide)
     )
@@
       (effects (font (size 1.27 1.27)) hide)
     )
-    (property "OEPS PN" "??" (at 139.7 59.69 0)
+    (property "OEPS PN" "-" (at 139.7 59.69 0)
       (effects (font (size 1.27 1.27)) hide)
     )
@@
     (pin "5")
     (pin "6")
+    (property "MPN" "-" (at 139.7 59.69 0)
+      (effects (font (size 1.27 1.27)) hide)
+    )
+    (property "Type" "-" (at 139.7 59.69 0)
+      (effects (font (size 1.27 1.27)) hide)
+    )
     (instances
       (project "headstage-neuropix2e"
@@
       (effects (font (size 1.27 1.27)) hide)
     )
-    (property "OEPS PN" "??" (at 160.02 110.49 0)
+    (property "OEPS PN" "OEPS010035" (at 160.02 110.49 0)
+      (effects (font (size 1.27 1.27)) hide)
+    )
+    (property "MPN" "GRM033R61E104KE14J" (at 160.02 110.49 0)
+      (effects (font (size 1.27 1.27)) hide)
+    )
+    (property "Type" "SMD" (at 160.02 110.49 0)
       (effects (font (size 1.27 1.27)) hide)
     )
@@
       (effects (font (size 1.27 1.27)) hide)
     )
-    (property "OEPS PN" "??" (at 149.86 144.78 0)
+    (property "OEPS PN" "OEPS010035" (at 149.86 144.78 0)
+      (effects (font (size 1.27 1.27)) hide)
+    )
+    (property "MPN" "GRM033R61E104KE14J" (at 149.86 144.78 0)
+      (effects (font (size 1.27 1.27)) hide)
+    )
+    (property "Type" "SMD" (at 149.86 144.78 0)
       (effects (font (size 1.27 1.27)) hide)
     )
@@
       (effects (font (size 1.27 1.27)) hide)
     )
-    (property "OEPS PN" "??" (at 96.52 58.42 0)
-      (effects (font (size 1.27 1.27)) hide)
-    )
+    (property "OEPS PN" "OEPS070030" (at 96.52 58.42 0)
+      (effects (font (size 1.27 1.27)) hide)
+    )
+    (property "MPN" "SBH11-PBPC-D05-ST-BK" (at 96.52 58.42 0)
+      (effects (font (size 1.27 1.27)) hide)
+    )
+    (property "Type" "TH" (at 96.52 58.42 0)
+      (effects (font (size 1.27 1.27)) hide)
+    )

Commit message: Corrected MPN of J6.
Parts:
- J6: MPN (none) -> 5050700622; Type (none) -> SMD
Changed lines of the file:
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@@
     (pin "MP3")
     (pin "MP4")
+    (property "MPN" "5050700622" (at 214.63 125.73 0)
+      (effects (font (size 1.27 1.27)) hide)
+    )
+    (property "Type" "SMD" (at 214.63 125.73 0)
+      (effects (font (size 1.27 1.27)) hide)
+    )
     (instances
       (project "headstage-neuropix2e"
