File: pcb-beta/perpherials.kicad_sch (KiCad schematic)
At the start: 9 parts, among them J4 TC2030, J6 050700622, J6 SBH11-PBPC-D05-ST-BK, U6 CAT24C04C4ATR, U7 BNO055

Commit message: Move pcb to pcb-beta directory
- Because this board only works with Beta-test NP2.0 probes
Parts:
- U6: value CAT24C04C4ATR -> M24C64-FCS6TP/K; footprint jonnew:ONSEMI_567JZ_WLCSP4-0.84x0.86 -> jonnew:ST_WLCSP5-0.959x1.073; symbol jonnew:CAT24Cxx -> jonnew:24Cxx-WC
Connections:
- net GPIO is gone; now on net +2V5: J6.6 (Pin_6)
- net GND: now also U6.A3 (VSS), U6.C1 (~{WC}); no longer U6.A2 (VSS)
- net SCL: now also U6.C3 (SCL); no longer U6.B1 (SCL)
Other:
- note added: "NB: This might need to be potted. UV light will erase."
- moved on the sheet: C25
